File: next_plate/next_plate.kicad_pcb (KiCad board)
At the start: 2 copper layers, 353.8 x 104.1 mm, 4 parts

Commit message: V2
Parts:
- removed FC660c_small_hole (x3): , Keyboard_Footprints:FC660c_small_hole
- added Plate_Cutout_Alps: , Keyboard_Footprints:Plate_Cutout_Alps, F.Cu at (281.0, 76.2)
- added Plate_Cutout_Alps: , Keyboard_Footprints:Plate_Cutout_Alps, F.Cu at (57.1, 57.1)
- added Plate_Cutout_Alps: , Keyboard_Footprints:Plate_Cutout_Alps, F.Cu at (366.7, 114.3)
- added Plate_Cutout_Alps: , Keyboard_Footprints:Plate_Cutout_Alps, F.Cu at (95.2, 57.1)
- added Plate_Cutout_Alps: , Keyboard_Footprints:Plate_Cutout_Alps, F.Cu at (76.2, 38.1)
- added Plate_Cutout_Alps: , Keyboard_Footprints:Plate_Cutout_Alps, F.Cu at (66.7, 114.3)
- added Plate_Cutout_Alps: , Keyboard_Footprints:Plate_Cutout_Alps, F.Cu at (214.3, 95.2)
- added Plate_Cutout_Alps: , Keyboard_Footprints:Plate_Cutout_Alps, F.Cu at (57.1, 38.1)
- added Plate_Cutout_Alps: , Keyboard_Footprints:Plate_Cutout_Alps, F.Cu at (223.8, 76.2)
- added Plate_Cutout_Alps: , Keyboard_Footprints:Plate_Cutout_Alps, F.Cu at (366.7, 38.1)
- added Plate_Cutout_Alps: , Keyboard_Footprints:Plate_Cutout_Alps, F.Cu at (76.2, 95.2)
- added Plate_Cutout_Alps: , Keyboard_Footprints:Plate_Cutout_Alps, F.Cu at (119.1, 57.1)
- added Plate_Cutout_Alps: , Keyboard_Footprints:Plate_Cutout_Alps, F.Cu at (204.8, 76.2)
- added Plate_Cutout_Alps: , Keyboard_Footprints:Plate_Cutout_Alps, F.Cu at (300.0, 76.2)
- added Plate_Cutout_Alps: , Keyboard_Footprints:Plate_Cutout_Alps, F.Cu at (228.6, 38.1)
- added Plate_Cutout_Alps: , Keyboard_Footprints:Plate_Cutout_Alps, F.Cu at (276.2, 57.1)
- added Plate_Cutout_Alps: , Keyboard_Footprints:Plate_Cutout_Alps, F.Cu at (290.5, 95.2)
- added Plate_Cutout_Alps: , Keyboard_Footprints:Plate_Cutout_Alps, F.Cu at (371.5, 57.1)
- added Plate_Cutout_Alps: , Keyboard_Footprints:Plate_Cutout_Alps, F.Cu at (233.4, 95.2)
- added Plate_Cutout_Alps: , Keyboard_Footprints:Plate_Cutout_Alps, F.Cu at (147.6, 114.3)
- added Plate_Cutout_Alps: , Keyboard_Footprints:Plate_Cutout_Alps, F.Cu at (181.0, 57.1)
- added Plate_Cutout_Alps: , Keyboard_Footprints:Plate_Cutout_Alps, F.Cu at (285.8, 38.1)
- added Plate_Cutout_Alps: , Keyboard_Footprints:Plate_Cutout_Alps, F.Cu at (95.2, 114.3)
- added Plate_Cutout_Alps: , Keyboard_Footprints:Plate_Cutout_Alps, F.Cu at (76.2, 57.1)
- added Plate_Cutout_Alps: , Keyboard_Footprints:Plate_Cutout_Alps, F.Cu at (147.6, 76.2)
- added Plate_Cutout_Alps: , Keyboard_Footprints:Plate_Cutout_Alps, F.Cu at (185.7, 76.2)
- added Plate_Cutout_Alps: , Keyboard_Footprints:Plate_Cutout_Alps, F.Cu at (257.2, 57.1)
- added Plate_Cutout_Alps: , Keyboard_Footprints:Plate_Cutout_Alps, F.Cu at (271.5, 95.2)
- added Plate_Cutout_Alps: , Keyboard_Footprints:Plate_Cutout_Alps, F.Cu at (38.1, 38.1)
- added Plate_Cutout_Alps: , Keyboard_Footprints:Plate_Cutout_Alps, F.Cu at (157.2, 95.2)
- added Plate_Cutout_Alps: , Keyboard_Footprints:Plate_Cutout_Alps, F.Cu at (161.9, 57.1)
- added Plate_Cutout_Alps: , Keyboard_Footprints:Plate_Cutout_Alps, F.Cu at (219.1, 57.1)
- added Plate_Cutout_Alps: , Keyboard_Footprints:Plate_Cutout_Alps, F.Cu at (266.7, 38.1)
- added Plate_Cutout_Alps: , Keyboard_Footprints:Plate_Cutout_Alps, F.Cu at (38.1, 57.1)
- added Plate_Cutout_Alps: , Keyboard_Footprints:Plate_Cutout_Alps, F.Cu at (190.5, 38.1)
- added Plate_Cutout_Alps: , Keyboard_Footprints:Plate_Cutout_Alps, F.Cu at (314.3, 57.1)
- added Plate_Cutout_Alps: , Keyboard_Footprints:Plate_Cutout_Alps, F.Cu at (247.7, 38.1)
- added Plate_Cutout_Alps: , Keyboard_Footprints:Plate_Cutout_Alps, F.Cu at (126.2, 95.2)
- added Plate_Cutout_Alps: , Keyboard_Footprints:Plate_Cutout_Alps, F.Cu at (95.2, 38.1)
- added Plate_Cutout_Alps: , Keyboard_Footprints:Plate_Cutout_Alps, F.Cu at (195.3, 95.2)
- added Plate_Cutout_Alps: , Keyboard_Footprints:Plate_Cutout_Alps, F.Cu at (152.4, 38.1)
- added Plate_Cutout_Alps: , Keyboard_Footprints:Plate_Cutout_Alps, F.Cu at (57.1, 76.2)
- added Plate_Cutout_Alps: , Keyboard_Footprints:Plate_Cutout_Alps, F.Cu at (171.4, 38.1)
- added Plate_Cutout_Alps: , Keyboard_Footprints:Plate_Cutout_Alps, F.Cu at (304.8, 38.1)
- added Plate_Cutout_Alps: , Keyboard_Footprints:Plate_Cutout_Alps, F.Cu at (352.4, 57.1)
- added Plate_Cutout_Alps: , Keyboard_Footprints:Plate_Cutout_Alps, F.Cu at (121.4, 76.2)
- added Plate_Cutout_Alps: , Keyboard_Footprints:Plate_Cutout_Alps, F.Cu at (319.1, 76.2)
- added Plate_Cutout_Alps: , Keyboard_Footprints:Plate_Cutout_Alps, F.Cu at (309.6, 95.2)
- added Plate_Cutout_Alps: , Keyboard_Footprints:Plate_Cutout_Alps, F.Cu at (342.9, 38.1)
- added Plate_Cutout_Alps: , Keyboard_Footprints:Plate_Cutout_Alps, F.Cu at (295.3, 57.1)
- added Plate_Cutout_Alps: , Keyboard_Footprints:Plate_Cutout_Alps, F.Cu at (76.2, 76.2)
- added Plate_Cutout_Alps: , Keyboard_Footprints:Plate_Cutout_Alps, F.Cu at (338.1, 114.3)
- added Plate_Cutout_Alps: , Keyboard_Footprints:Plate_Cutout_Alps, F.Cu at (364.3, 76.2)
- added Plate_Cutout_Alps: , Keyboard_Footprints:Plate_Cutout_Alps, F.Cu at (252.4, 95.2)
- added Plate_Cutout_Alps: , Keyboard_Footprints:Plate_Cutout_Alps, F.Cu at (323.9, 38.1)
- added Plate_Cutout_Alps: , Keyboard_Footprints:Plate_Cutout_Alps, F.Cu at (119.1, 114.3)
- added Plate_Cutout_Alps: , Keyboard_Footprints:Plate_Cutout_Alps, F.Cu at (209.6, 38.1)
- added Plate_Cutout_Alps: , Keyboard_Footprints:Plate_Cutout_Alps, F.Cu at (114.3, 38.1)
- added Plate_Cutout_Alps: , Keyboard_Footprints:Plate_Cutout_Alps, F.Cu at (38.1, 76.2)
- added Plate_Cutout_Alps: , Keyboard_Footprints:Plate_Cutout_Alps, F.Cu at (133.3, 38.1)
- added Plate_Cutout_Alps: , Keyboard_Footprints:Plate_Cutout_Alps, F.Cu at (176.2, 95.2)
- added Plate_Cutout_Alps: , Keyboard_Footprints:Plate_Cutout_Alps, F.Cu at (242.9, 76.2)
- added Plate_Cutout_Alps: , Keyboard_Footprints:Plate_Cutout_Alps, F.Cu at (166.7, 76.2)
- added Plate_Cutout_Alps: , Keyboard_Footprints:Plate_Cutout_Alps, F.Cu at (261.9, 76.2)
- added Plate_Cutout_Alps: , Keyboard_Footprints:Plate_Cutout_Alps, F.Cu at (359.6, 95.2)
- added Plate_Cutout_Alps: , Keyboard_Footprints:Plate_Cutout_Alps, F.Cu at (338.1, 76.2)
- added Plate_Cutout_Alps: , Keyboard_Footprints:Plate_Cutout_Alps, F.Cu at (95.2, 76.2)
- added Plate_Cutout_Alps: , Keyboard_Footprints:Plate_Cutout_Alps, F.Cu at (333.4, 57.1)
- added Plate_Cutout_Alps: , Keyboard_Footprints:Plate_Cutout_Alps, F.Cu at (238.1, 57.1)
- added Plate_Cutout_Alps: , Keyboard_Footprints:Plate_Cutout_Alps, F.Cu at (328.6, 95.2)
- added Plate_Cutout_Alps: , Keyboard_Footprints:Plate_Cutout_Alps, F.Cu at (200.0, 57.1)
- added Plate_Cutout_Alps: , Keyboard_Footprints:Plate_Cutout_Alps, F.Cu at (57.1, 95.2)
- added Plate_Cutout_Alps: , Keyboard_Footprints:Plate_Cutout_Alps, F.Cu at (142.9, 57.1)
- added Plate_Cutout_Alps: , Keyboard_Footprints:Plate_Cutout_Alps, F.Cu at (95.2, 95.2)
- added Plate_Cutout_Alps: , Keyboard_Footprints:Plate_Cutout_Alps, F.Cu at (38.1, 104.8)
- Plate_Cutout_Alps: renamed from ?; value SKCM_Plate Cutout -> (none); footprint Keyboard_Footprints:SKCM_Plate_Cutout -> Keyboard_Footprints:Plate_Cutout_Alps
Other:
- outline, holes or cut-outs redrawn
- net class Default removed
- rule pad_to_mask_clearance: 0.2 -> 0

Commit message: Numpad Config Changed
Parts:
- moved Plate_Cutout_Alps 38.1 mm to (57.1, 114.3)
- moved Plate_Cutout_Alps 19.0 mm to (85.7, 114.3)
Other:
- outline, holes or cut-outs redrawn
Changed lines of the file:
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@@
   )
   (footprint "Keyboard_Footprints:Plate_Cutout_Alps" (layer "F.Cu")
-    (at 66.675 114.3)
+    (at 85.725 114.3)
     (attr through_hole)
     (fp_text reference "Plate_Cutout_Alps" (at 0 0.5) (layer "F.SilkS") hide
@@
   )
   (footprint "Keyboard_Footprints:Plate_Cutout_Alps" (layer "F.Cu")
-    (at 95.25 114.3)
+    (at 57.15 114.3)
     (attr through_hole)
     (fp_text reference "Plate_Cutout_Alps" (at 0 0.5) (layer "F.SilkS") hide
@@
   (gr_line (start 300.1375 124.5) (end 209.4375 124.5) (layer "Edge.Cuts") (width 0.01))
   (gr_line (start 105.9875 24.15) (end 105.9875 24.65) (layer "Edge.Cuts") (width 0.01))
-  (gr_line (start 51.275 118.15) (end 51.275 123.25) (layer "Edge.Cuts") (width 0.01))
+  (gr_line (start 70.325 118.15) (end 70.325 123.25) (layer "Edge.Cuts") (width 0.01))
   (gr_line (start 305.9875 25.4) (end 305.9875 24.15) (layer "Edge.Cuts") (width 0.01))
   (gr_circle (center 204.7875 114.3) (end 207.9125 114.3) (layer "Edge.Cuts") (width 0.01) (fill none))
@@
   (gr_line (start 197.7125 115.4) (end 197.7125 113.2) (layer "Edge.Cuts") (width 0.01))
   (gr_line (start 211.8625 115.4) (end 209.6625 115.4) (layer "Edge.Cuts") (width 0.01))
-  (gr_line (start 53.875 118.15) (end 51.275 118.15) (layer "Edge.Cuts") (width 0.01))
+  (gr_line (start 72.925 118.15) (end 70.325 118.15) (layer "Edge.Cuts") (width 0.01))
   (gr_line (start 353.5 118.5) (end 357.5 118.5) (layer "Edge.Cuts") (width 0.1))
   (gr_arc (start 203.5875 127) (mid 204.7875 125.8) (end 205.9875 127) (layer "Edge.Cuts") (width 0.01))
@@
   (gr_line (start 180.4875 118.15) (end 180.4875 123.25) (layer "Edge.Cuts") (width 0.01))
   (gr_line (start 206.5875 24.15) (end 209.4375 27.9) (layer "Edge.Cuts") (width 0.01))
-  (gr_line (start 51.275 123.25) (end 53.875 123.25) (layer "Edge.Cuts") (width 0.01))
+  (gr_line (start 70.325 123.25) (end 72.925 123.25) (layer "Edge.Cuts") (width 0.01))
   (gr_arc (start 27.9 28.9) (mid 28.192893 28.192893) (end 28.9 27.9) (layer "Edge.Cuts") (width 0.01))
   (gr_line (start 105.9875 127) (end 105.9875 127.75) (layer "Edge.Cuts") (width 0.01))
@@
   (gr_line (start 183.0875 123.25) (end 183.0875 118.15) (layer "Edge.Cuts") (width 0.01))
   (gr_line (start 183.0875 110.45) (end 180.4875 110.45) (layer "Edge.Cuts") (width 0.01))
-  (gr_line (start 82.075 118.15) (end 82.075 123.25) (layer "Edge.Cuts") (width 0.01))
+  (gr_line (start 101.125 118.15) (end 101.125 123.25) (layer "Edge.Cuts") (width 0.01))
   (gr_line (start 180.4875 105.35) (end 183.0875 105.35) (layer "Edge.Cuts") (width 0.01))
   (gr_line (start 132.14375 80.05) (end 134.74375 80.05) (layer "Edge.Cuts") (width 0.01))
   (gr_line (start 343.46875 86.3) (end 340.86875 86.3) (layer "Edge.Cuts") (width 0.01))
   (gr_line (start 276.1125 115.4) (end 276.1125 113.2) (layer "Edge.Cuts") (width 0.01))
-  (gr_line (start 79.475 118.15) (end 82.075 118.15) (layer "Edge.Cuts") (width 0.01))
+  (gr_line (start 98.525 118.15) (end 101.125 118.15) (layer "Edge.Cuts") (width 0.01))
   (gr_line (start 110.10625 91.4) (end 110.10625 86.3) (layer "Edge.Cuts") (width 0.01))
   (gr_line (start 285.8625 115.4) (end 288.0625 115.4) (layer "Edge.Cuts") (width 0.01))
@@
   (gr_line (start 302.6875 118.15) (end 305.2875 118.15) (layer "Edge.Cuts") (width 0.01))
   (gr_arc (start 103.5875 127) (mid 104.7875 125.8) (end 105.9875 127) (layer "Edge.Cuts") (width 0.01))
-  (gr_line (start 53.875 123.25) (end 53.875 118.15) (layer "Edge.Cuts") (width 0.01))
+  (gr_line (start 72.925 123.25) (end 72.925 118.15) (layer "Edge.Cuts") (width 0.01))
   (gr_line (start 302.9875 128.25) (end 300.1375 124.5) (layer "Edge.Cuts") (width 0.01))
   (gr_line (start 375.66875 86.3) (end 378.26875 86.3) (layer "Edge.Cuts") (width 0.01))
@@
   (gr_line (start 180.4875 123.25) (end 183.0875 123.25) (layer "Edge.Cuts") (width 0.01))
   (gr_line (start 303.5875 127) (end 303.5875 128.25) (layer "Edge.Cuts") (width 0.01))
-  (gr_line (start 79.475 123.25) (end 79.475 118.15) (layer "Edge.Cuts") (width 0.01))
+  (gr_line (start 98.525 123.25) (end 98.525 118.15) (layer "Edge.Cuts") (width 0.01))
   (gr_line (start 102.9875 128.25) (end 103.5875 128.25) (layer "Edge.Cuts") (width 0.01))
   (gr_line (start 134.74375 85.15) (end 132.14375 85.15) (layer "Edge.Cuts") (width 0.01))
@@
   (gr_line (start 305.2875 105.35) (end 305.2875 110.45) (layer "Edge.Cuts") (width 0.01))
   (gr_line (start 200.1375 124.5) (end 109.4375 124.5) (layer "Edge.Cuts") (width 0.01))
-  (gr_line (start 82.075 123.25) (end 79.475 123.25) (layer "Edge.Cuts") (width 0.01))
+  (gr_line (start 101.125 123.25) (end 98.525 123.25) (layer "Edge.Cuts") (width 0.01))
   (gr_line (start 202.9875 128.25) (end 203.5875 128.25) (layer "Edge.Cuts") (width 0.01))
   (gr_arc (start 105.9875 25.4) (mid 104.7875 26.6) (end 103.5875 25.4) (layer "Edge.Cuts") (width 0.01))

Commit message: Added LED opttion
Other:
- outline, holes or cut-outs redrawn
Changed lines of the file:
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@@
   (gr_line (start 183.0875 123.25) (end 183.0875 118.15) (layer "Edge.Cuts") (width 0.01))
   (gr_line (start 183.0875 110.45) (end 180.4875 110.45) (layer "Edge.Cuts") (width 0.01))
+  (gr_circle (center 95.25 47.625) (end 97.25 47.625) (layer "Edge.Cuts") (width 0.1) (fill none))
   (gr_line (start 101.125 118.15) (end 101.125 123.25) (layer "Edge.Cuts") (width 0.01))
   (gr_line (start 180.4875 105.35) (end 183.0875 105.35) (layer "Edge.Cuts") (width 0.01))
